File: lora-pcb.kicad/lora-pcb.kicad_sch (KiCad schematic)
At the start: 10 parts, among them J1 Conn_SUR, J2 Conn_THT, U1 RFM95W-868S2

Commit message: LoRa-PCB Rev 1.00: version with 433MHz (ready for production)
Parts:
- U1: LCSC C2844472 -> C2844474
Changed lines of the file:
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@@
   (title_block
     (title "LoRa PCB with SURS-Connector")
-    (date "2024-02-07")
-    (rev "0.9")
+    (date "2024-02-22")
+    (rev "1.0")
     (company "Bernhard Bablok")
     (comment 1 "https://github.com/bablokb/pcb-pico-datalogger")
@@
       (effects (font (size 1.27 1.27)) hide)
     )
-    (property "LCSC" "C2844472" (id 4) (at 163.068 46.736 0)
-      (effects (font (size 1.27 1.27)) hide)
-    )
+    (property "LCSC" "C2844474" (id 4) (at 163.068 46.736 0)
+      (effects (font (size 1.27 1.27)) hide)
+    )
